File: pcb/air_poll.kicad_sch (KiCad schematic)
At the start: 0 parts

Commit message: Fix: Standardize backend API URLs to 127.0.0.1 from localhost
Parts:
- added C1, C2: 100n, e-radionica.com footprinti:0603C, symbol e-radionica.com schematics:0603C
- added D1: purple, e-radionica.com footprinti:0402LED, symbol e-radionica.com schematics:0402LED
- added K1: HEADER_MALE_4X1, e-radionica.com footprinti:HEADER_MALE_4X1, symbol e-radionica.com schematics:HEADER_MALE_4X1
- added R1, R3: 10k, e-radionica.com footprinti:0603R, symbol e-radionica.com schematics:0603R
- added R2: TC33X-2-103E, e-radionica.com footprinti:tc33x-2-103e, symbol e-radionica.com schematics:tc33x-2-103e
- added R4: 2k2, e-radionica.com footprinti:0402R, symbol e-radionica.com schematics:0402R
- added U1: DOIT-ESP32-DEVKIT-V1, symbol esp:DOIT-ESP32-DEVKIT-V1
- added U2: PMS5003, PMS5003:PMS5003, symbol air_poll:PMS5003
- added U3: BME280, BME280:PSON65P250X250X100-8N, symbol air_poll:BME280
- added U4: MQ-X, e-radionica.com footprinti:MQ, symbol e-radionica.com schematics:MQ
- added U5: LM393, e-radionica.com footprinti:SOIC−8, symbol e-radionica.com schematics:LM393
Connections:
- new net: D1.1 (A), R4.2
- new net 5V: C2.2, K1.4, R2.1, R3.2, U4.1 (A), U4.2 (H), U4.3 (A), U5.8 (VCC)
- new net AO: C1.2, K1.2, R1.2, U4.4 (B), U4.6 (B), U5.3 (1_IN+)
- new net D0: K1.3, R3.1, R4.1, U5.1 (1_OUT)
- new net GND: C1.1, C2.1, D1.2 (K), K1.1, R1.1, R2.3, U3.1 (GND), U3.7 (GND), U4.5 (H), U5.4 (GND)
- new net POT: R2.2, U5.2 (1_IN-)
Other:
- note added: "LM393"
